File: power_usb.kicad_sch (KiCad schematic)
At the start: 33 parts, among them J1 USB_C_Receptacle, U1 LP2985-3.3, U3 CP2102N-A02-GQFN24, U5 LP2985-3.3

Commit message: UPDI: replicate EtherKeyerMini UPDI circuit (J5/R13/D4/D5/JP1/JP2); remove CP2102N LEDs D2/D3 + R10/R11, NC pins 13/14
Parts:
- removed D2: RED, LED_SMD:LED_0603_1608Metric, symbol Device:LED_Small
- removed D3: BLUE, LED_SMD:LED_0603_1608Metric, symbol Device:LED_Small
- removed R10: 470, Resistor_SMD:R_0603_1608Metric, symbol Device:R_Small
- removed R11: 330, Resistor_SMD:R_0603_1608Metric, symbol Device:R_Small
Connections:
- net LED_RXT: no longer names the net of U3.13 (~{RXT}/GPIO.1)
- net LED_TXT: no longer names the net of U3.14 (~{TXT}/GPIO.0)
- no-connect marks 11 -> 13

Commit message: Wire local connections (labels only for long/cross-sheet runs); +3V3_MCU diode-OR rail (D6/D5); drop UPDI JP1/JP2; fix C14 fields
Connections:
- net CC1: no longer names the net of J1.A5 (CC1), R1.1
- net CC2: no longer names the net of J1.B5 (CC2), R2.1
- net OLED_LDO_OUT: no longer names the net of C9.1, FB2.1, U5.5 (VOUT)
- net U1_BP: no longer names the net of C2.1, U1.4 (BP)
- net U5_BP: no longer names the net of C8.1, U5.4 (BP)
