File: synth_rf.kicad_sch (KiCad schematic)
At the start: 60 parts, among them J2 SMA CLK0, J3 SMA CLK1, J4 SMA CLK2, U2 Si5351A-B-GT, X1 25MHz TCXO

Commit message: Wire local connections (labels only for long/cross-sheet runs); +3V3_MCU diode-OR rail (D6/D5); drop UPDI JP1/JP2; fix C14 fields
Parts:
- R27: VERIFY I2C pull-up value not fixed (PLAN 2.2-4.7k); no LCSC chosen. -> I2C pull-up value not fixed (PLAN 2.2-4.7k); no LCSC chosen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
Connections:
- net +3V3_CLK: no longer R27.1, R28.1
- net CLK0_DC: no longer names the net of C100.2, R101.1, R102.1, R104.1
- net CLK0_F1: no longer names the net of C101.1, C105.1, L1.1, R102.2
- net CLK0_F2: no longer names the net of C102.1, C105.2, C106.1, L1.2, L2.1
- net CLK0_F3: no longer names the net of C103.1, C106.2, C107.1, L2.2, L3.1
- net CLK0_F4: no longer names the net of C104.1, C107.2, L3.2, R103.1
- net CLK0_OUT: no longer names the net of J2.1 (In), R103.2, R104.2
- net CLK0_S: no longer names the net of C100.1, R100.2
- net CLK1_DC: no longer names the net of C120.2, R121.1, R122.1, R124.1
- net CLK1_F1: no longer names the net of C121.1, C125.1, L4.1, R122.2
- net CLK1_F2: no longer names the net of C122.1, C125.2, C126.1, L4.2, L5.1
- net CLK1_F3: no longer names the net of C123.1, C126.2, C127.1, L5.2, L6.1
- net CLK1_F4: no longer names the net of C124.1, C127.2, L6.2, R123.1
- net CLK1_OUT: no longer names the net of J3.1 (In), R123.2, R124.2
- net CLK1_S: no longer names the net of C120.1, R120.2
- net CLK2_DC: no longer names the net of C140.2, R141.1, R142.1, R144.1
- net CLK2_F1: no longer names the net of C141.1, C145.1, L7.1, R142.2
- net CLK2_F2: no longer names the net of C142.1, C145.2, C146.1, L7.2, L8.1
- net CLK2_F3: no longer names the net of C143.1, C146.2, C147.1, L8.2, L9.1
- net CLK2_F4: no longer names the net of C144.1, C147.2, L9.2, R143.1
- net CLK2_OUT: no longer names the net of J4.1 (In), R143.2, R144.2
- net CLK2_S: no longer names the net of C140.1, R140.2
- net SI_XA: no longer names the net of C6.2, U2.2 (XA)
- net TCXO_EN: no longer names the net of R6.2, X1.1 (NC/EN)
- net TCXO_OUT: no longer names the net of C6.1, X1.3 (OUT)
- net TCXO_VDD: no longer names the net of C5.1, R5.2, R6.1, X1.4 (VDD)
- new net +3V3_MCU: R27.1, R28.1
Other:
- note added: "VERIFY (unconfirmed items on this sheet): - X1: TCXO stock thin (718); buy before ordering. - R27: I2C pull-up value not fixed (PLAN 2.2-4.7k); no LCSC chosen. Pulled to +3V3_MCU (not +3V3_CLK) so SCL/SDA never exceed ATtiny VDD; Si5351 VIH 0.7*VDD=2.31 V vs ~2.95 V high - check. - R28: as R27 - R100: 0603 0R series (Jason decision); LCSC code not in PLAN (C17477 is 0805). - C100: DC-block LF cor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"
- note removed: "VERIFY (unconfirmed items on this sheet): - X1: TCXO stock thin (718); buy before ordering. - R27: I2C pull-up value not fixed (PLAN 2.2-4.7k); no LCSC chosen. - R28: as R27 - R100: 0603 0R series (Jason decision); LCSC code not in PLAN (C17477 is 0805). - C100: DC-block LF corner ~32 kHz into 50 ohm (PLAN Q6). - R101: DNP shunt ~120 ohm back-match of ~85 ohm source (datasheet Zo); part/LCSC not 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"

Commit message: Drop +3V3_MCU/D5/D6: U4 and pull-ups back on +3V3D; J5 pin 1 = +3V3D VCC reference (USB-powered programming)
Parts:
- R27: VERIFY I2C pull-up value not fixed (PLAN 2.2-4.7k); no LCSC chosen. Pulled to +3V3_MCU (not +3V3_CLK) so SCL/SDA never exceed ATtiny VDD; Si5351 VIH 0.7*VDD=2.31 V vs ~2.95 V high - check. -> I2C pull-up value not fixed (PLAN 2.2-4.7k); no LCSC chosen. On +3V3D: ATtiny, Si5351, CP2102N and OLED all at 3.3 V, so I2C levels match.
Connections:
- net +3V3_MCU renamed +3V3D
Other:
- note added: "VERIFY (unconfirmed items on this sheet): - X1: TCXO stock thin (718); buy before ordering. - R27: I2C pull-up value not fixed (PLAN 2.2-4.7k); no LCSC chosen. On +3V3D: ATtiny, Si5351, CP2102N and OLED all at 3.3 V, so I2C levels match. - R28: as R27 - R100: 0603 0R series (Jason decision); LCSC code not in PLAN (C17477 is 0805). - C100: DC-block LF corner ~32 kHz into 50 ohm (PLAN Q6). - R101: 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"
- note removed: "VERIFY (unconfirmed items on this sheet): - X1: TCXO stock thin (718); buy before ordering. - R27: I2C pull-up value not fixed (PLAN 2.2-4.7k); no LCSC chosen. Pulled to +3V3_MCU (not +3V3_CLK) so SCL/SDA never exceed ATtiny VDD; Si5351 VIH 0.7*VDD=2.31 V vs ~2.95 V high - check. - R28: as R27 - R100: 0603 0R series (Jason decision); LCSC code not in PLAN (C17477 is 0805). - C100: DC-block LF cor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"

Commit message: synth_rf: populate Cauer LPFs (CLK0/1 60 MHz, CLK2 160 MHz) with LCSC parts; replace 0R filter links with solder jumpers (JP1x2/JP1x3 NC in-line, JP1x4 NO bypass); interchangeability note
Parts:
- removed R102, R103, R104, R122, R123, R124, R142, R143, R144: 0, Resistor_SMD:R_0805_2012Metric, symbol Device:R_Small
- added JP102, JP103, JP122, JP123, JP142, JP143: NC, Jumper:SolderJumper-2_P1.3mm_Bridged_RoundedPad1.0x1.5mm, symbol Jumper:SolderJumper_2_Bridged
- added JP104, JP124, JP144: NO, Jumper:SolderJumper-2_P1.3mm_Open_RoundedPad1.0x1.5mm, symbol Jumper:SolderJumper_2_Open
- C101: value DNP -> 33p; footprint Capacitor_SMD:C_0805_2012Metric -> Capacitor_SMD:C_0603_1608Metric; LCSC (none) -> C519485; MPN (none) -> CC0603FRNPO9BN330; Manufacturer (none) -> YAGEO; VERIFY LPF values builder choice (DNP) -> (none); now fitted
- C102, C122: value DNP -> 75p; footprint Capacitor_SMD:C_0805_2012Metric -> Capacitor_SMD:C_0603_1608Metric; LCSC (none) -> C519496; MPN (none) -> CC0603FRNPO9BN750; Manufacturer (none) -> YAGEO; now fitted
- C103, C123: value DNP -> 82p; footprint Capacitor_SMD:C_0805_2012Metric -> Capacitor_SMD:C_0603_1608Metric; LCSC (none) -> C519487; MPN (none) -> CC0603FRNPO9BN820; Manufacturer (none) -> YAGEO; now fitted
- C104, C124: value DNP -> 43p; footprint Capacitor_SMD:C_0805_2012Metric -> Capacitor_SMD:C_0603_1608Metric; LCSC (none) -> C519493; MPN (none) -> CC0603FRNPO9BN430; Manufacturer (none) -> YAGEO; now fitted
- C105: value DNP -> 39p; footprint Capacitor_SMD:C_0805_2012Metric -> Capacitor_SMD:C_0603_1608Metric; LCSC (none) -> C527048; MPN (none) -> CC0603FRNPO9BN390; Manufacturer (none) -> YAGEO; VERIFY Parallel C across L (elliptic) per LowPassFilterModule - un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 -> 9.1p only +/-0.25pF in stock (C513588); 24p +/-2% stock thi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; now fitted
- C106, C126: value DNP -> 20p; footprint Capacitor_SMD:C_0805_2012Metric -> Capacitor_SMD:C_0603_1608Metric; LCSC (none) -> C326779; MPN (none) -> CC0603FRNPO9BN200; Manufacturer (none) -> YAGEO; now fitted
- C107, C127: value DNP -> 9.1p; footprint Capacitor_SMD:C_0805_2012Metric -> Capacitor_SMD:C_0603_1608Metric; LCSC (none) -> C513588; MPN (none) -> CC0603CRNPO9BN9R1; Manufacturer (none) -> YAGEO; now fitted
- C121: value DNP -> 33p; footprint Capacitor_SMD:C_0805_2012Metric -> Capacitor_SMD:C_0603_1608Metric; LCSC (none) -> C519485; MPN (none) -> CC0603FRNPO9BN330; Manufacturer (none) -> YAGEO; now fitted
- C125: value DNP -> 39p; footprint Capacitor_SMD:C_0805_2012Metric -> Capacitor_SMD:C_0603_1608Metric; LCSC (none) -> C527048; MPN (none) -> CC0603FRNPO9BN390; Manufacturer (none) -> YAGEO; now fitted
- C141: value DNP -> 3.6p; footprint Capacitor_SMD:C_0805_2012Metric -> Capacitor_SMD:C_0603_1608Metric; LCSC (none) -> C519106; MPN (none) -> CC0603BRNPO9BN3R6; Manufacturer (none) -> YAGEO; now fitted
- C142: value DNP -> 24p; footprint Capacitor_SMD:C_0805_2012Metric -> Capacitor_SMD:C_0603_1608Metric; LCSC (none) -> C2857979; MPN (none) -> 0603CG240G500NT; Manufacturer (none) -> FH; now fitted
- C143: value DNP -> 30p; footprint Capacitor_SMD:C_0805_2012Metric -> Capacitor_SMD:C_0603_1608Metric; LCSC (none) -> C519491; MPN (none) -> CC0603FRNPO9BN300; Manufacturer (none) -> YAGEO; now fitted
- C144: value DNP -> 18p; footprint Capacitor_SMD:C_0805_2012Metric -> Capacitor_SMD:C_0603_1608Metric; LCSC (none) -> C527046; MPN (none) -> CC0603FRNPO9BN180; Manufacturer (none) -> YAGEO; now fitted
- C145: value DNP -> 16p; footprint Capacitor_SMD:C_0805_2012Metric -> Capacitor_SMD:C_0603_1608Metric; LCSC (none) -> C519489; MPN (none) -> CC0603FRNPO9BN160; Manufacturer (none) -> YAGEO; now fitted
- C146: value DNP -> 5.6p; footprint Capacitor_SMD:C_0805_2012Metric -> Capacitor_SMD:C_0603_1608Metric; LCSC (none) -> C519111; MPN (none) -> CC0603BRNPO9BN5R6; Manufacturer (none) -> YAGEO; now fitted
- C147: value DNP -> 2.0p; footprint Capacitor_SMD:C_0805_2012Metric -> Capacitor_SMD:C_0603_1608Metric; LCSC (none) -> C513620; MPN (none) -> CC0603BRNPO9BN2R0; Manufacturer (none) -> YAGEO; now fitted
- L1: value DNP -> 100n; footprint Inductor_SMD:L_0805_2012Metric -> Inductor_SMD:L_1008_2520Metric; LCSC (none) -> C1330579; MPN (none) -> LQW2UASR10G0CL; Manufacturer (none) -> Murata; VERIFY LPF inductor size (SMD vs T37 option, PLAN Q7) -> LQW2UAS stock 0.9-3.3k/part; buy ahead. 150n uses +/-1% C20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; now fitted
- L2, L3, L5, L6: value DNP -> 150n; footprint Inductor_SMD:L_0805_2012Metric -> Inductor_SMD:L_1008_2520Metric; LCSC (none) -> C2044861; MPN (none) -> LQW2UASR15F00L; Manufacturer (none) -> Murata; now fitted
- L4: value DNP -> 100n; footprint Inductor_SMD:L_0805_2012Metric -> Inductor_SMD:L_1008_2520Metric; LCSC (none) -> C1330579; MPN (none) -> LQW2UASR10G0CL; Manufacturer (none) -> Murata; now fitted
- L7: value DNP -> 33n; footprint Inductor_SMD:L_0805_2012Metric -> Inductor_SMD:L_1008_2520Metric; LCSC (none) -> C2043161; MPN (none) -> LQW2UAS33NG0CL; Manufacturer (none) -> Murata; now fitted
- L8, L9: value DNP -> 68n; footprint Inductor_SMD:L_0805_2012Metric -> Inductor_SMD:L_1008_2520Metric; LCSC (none) -> C703709; MPN (none) -> LQW2UAS68NG00L; Manufacturer (none) -> Murata; now fitted
Connections:
- net at J3.1 (In): now also JP123.2 (B), JP124.2 (B)
- net at C100.2, R101.1: now also JP102.1 (A), JP104.1 (A)
- net at C144.1, C147.2, L9.2: now also JP143.1 (A)
- net at C140.2, R141.1: now also JP142.1 (A), JP144.1 (A)
- net at J4.1 (In): now also JP143.2 (B), JP144.2 (B)
- net at C101.1, C105.1, L1.1: now also JP102.2 (B)
- net at C120.2, R121.1: now also JP122.1 (A), JP124.1 (A)
- net at C124.1, C127.2, L6.2: now also JP123.1 (A)
- net at J2.1 (In): now also JP103.2 (B), JP104.2 (B)
- net at C104.1, C107.2, L3.2: now also JP103.1 (A)
- net at C141.1, C145.1, L7.1: now also JP142.2 (B)
- net at C121.1, C125.1, L4.1: now also JP122.2 (B)
Other:
- note added: "Jumpers: JP102/JP103, JP122/JP123, JP142/JP143 in-line, normally closed (cut to remove filter). JP104/JP124/JP144 filter bypass, normally open (bridge after cutting in-line pair). Keep in-line jumper pads <=2 mm from junction (PLAN 6). Filter values are interchangeable per output (same footprint): CLK0/CLK1: 60 MHz Cauer (HF + 6 m; matched pair keeps quadrature phase). CLK2: 160 MHz Cauer. Not a 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"
- note added: "Si5351A + 25 MHz TCXO copied from Si5351A Breakout Rev F (R5/C5/C6/R6/C4, XB open). Each output: Rs 0R -> Cb 100n DC block -> DNP shunt -> 7th-order Cauer LPF between NC solder jumpers, NO bypass jumper -> SMA."
- note removed: "Bypass: RC (R104/R124/R144) fitted by default; RA/RB DNP. Filter build: fit RA/RB, remove RC. Keep RA/RB pads <=2 mm from junction (PLAN 6)."
- note removed: "Si5351A + 25 MHz TCXO copied from Si5351A Breakout Rev F (R5/C5/C6/R6/C4, XB open). Each output: Rs 0R -> Cb 100n DC block -> DNP shunt -> LPF (DNP) with 0R bypass -> SMA."
