File: PCB/power_usb.kicad_sch (KiCad schematic)
At the start: 38 parts, among them J1 USB_C_Receptacle, U1 LP2985-3.3, U3 CP2102N-A02-GQFN24, U5 LP2985-3.3

Commit message: R9: C110776 (YAGEO RT0603BRD071KL 0.1%) -> Basic C21190 (UNI-ROYAL 0603WAF1001T5E 1%), grouped with R29. Extended parts 33->32. ERC 0, DRC 15 accepted SMA hits, 0 unconnected/parity; fab + docs regenerated
Parts:
- R9: LCSC C110776 -> C21190; MPN RT0603BRD071KL -> 0603WAF1001T5E; Manufacturer YAGEO -> UNI-ROYAL
Changed lines of the file:
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@@
 			)
 		)
-		(property "LCSC" "C110776"
+		(property "LCSC" "C21190"
 			(at 137.16 59.69 0)
 			(hide yes)
@@
 			)
 		)
-		(property "MPN" "RT0603BRD071KL"
+		(property "MPN" "0603WAF1001T5E"
 			(at 137.16 59.69 0)
 			(hide yes)
@@
 			)
 		)
-		(property "Manufacturer" "YAGEO"
+		(property "Manufacturer" "UNI-ROYAL"
 			(at 137.16 59.69 0)
 			(hide yes)
