File: PCB/synth_rf.kicad_sch (KiCad schematic)
At the start: 66 parts, among them J2 SMA CLK0, J3 SMA CLK1, J4 SMA CLK2, U2 Si5351A-B-GT, X1 25MHz TCXO

Commit message: X1 TCXO pin 1 (NC/EN) tied to GND, R6 (VDD->pin 1) removed; same fix as OpenBeacon2 2de6f2e. PCB: R6 footprint and its VDD stub removed, X1.1 to GND via under X1, zones refilled. ERC 0, DRC 15 accepted SMA edge hits (unchanged), 0 unconnected/parity; docs + fab regenerated
Parts:
- removed R6: 0, Resistor_SMD:R_0805_2012Metric, symbol Device:R_Small_US
Connections:
- net GND: now also X1.1 (NC/EN)
Changed lines of the file:
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@@
 	(wire
 		(pts
-			(xy 59.69 72.39) (xy 44.45 72.39)
-		)
-		(stroke
-			(width 0)
-			(type default)
-		)
-	)
-	(wire
-		(pts
 			(xy 152.4 172.72) (xy 152.4 175.26)
 		)
@@
 	(wire
 		(pts
-			(xy 44.45 77.47) (xy 44.45 87.63)
+			(xy 44.45 87.63) (xy 44.45 90.17)
 		)
 		(stroke
@@
 	(symbol
 		(lib_id "power:GND")
+		(at 44.45 90.17 0)
+		(unit 1)
+		(body_style 1)
+		(exclude_from_sim no)
+		(in_bom no)
+		(on_board yes)
+		(in_pos_files yes)
+		(dnp no)
+		(property "Reference" "#PWR924"
+			(at 44.45 90.17 0)
+			(hide yes)
+			(show_name no)
+			(do_not_autoplace no)
+			(effects
+				(font
+					(size 1.27 1.27)
+				)
+			)
+		)
+		(property "Value" "GND"
+			(at 44.45 93.98 0)
+			(show_name no)
+			(do_not_autoplace no)
+			(effects
+				(font
+					(size 1.27 1.27)
+				)
+			)
+		)
+		(property "Footprint" ""
+			(at 44.45 90.17 0)
+			(hide yes)
+			(show_name no)
+			(do_not_autoplace no)
+			(effects
+				(font
+					(size 1.27 1.27)
+				)
+			)
+		)
+		(property "Datasheet" ""
+			(at 44.45 90.17 0)
+			(hide yes)
+			(show_name no)
+			(do_not_autoplace no)
+			(effects
+				(font
+					(size 1.27 1.27)
+				)
+			)
+		)
+		(property "Description" ""
+			(at 44.45 90.17 0)
+			(show_name no)
+			(do_not_autoplace no)
+			(effects
+				(font
+					(size 1.27 1.27)
+				)
+			)
+		)
+		(pin "1"
+		)
+		(instances
+			(project "Si5351AVFO"
+				(path "/a0000000-0000-4000-8000-000000000001/b0000000-0000-4000-8000-000000000004"
+					(reference "#PWR924")
+					(unit 1)
+				)
+			)
+		)
+	)
+	(symbol
+		(lib_id "power:GND")
 		(at 60.96 180.34 0)
 		(unit 1)
@@
 			)
 		)
-		(property "Description" "4-pin 3225 TCXO, clipped-sine output; pin 1 NC/EN (NC on fitted part; EN on active-high-enable TCXOs via DNP R6)"
+		(property "Description" "4-pin 3225 TCXO, clipped-sine output; pin 1 NC/EN, tied to GND (YXC 3225 pin 1 is NC: float or GND)"
 			(at 59.69 87.63 0)
 			(hide yes)
@@
 					(unit 1)
 				)
-			)
-		)
-	)
-	(symbol
-		(lib_id "Device:R_Small_US")
-		(at 44.45 74.93 0)
-		(unit 1)
-		(body_style 1)
-		(exclude_from_sim no)
-		(in_bom yes)
-		(on_board yes)
-		(in_pos_files yes)
-		(dnp yes)
-		(property "Reference" "R6"
-			(at 46.25 74.33 0)
-			(show_name no)
-			(do_not_autoplace no)
-			(effects
-				(font
-					(size 1.27 1.27)
-				)
-				(justify left)
-			)
-		)
-		(property "Value" "0"
-			(at 46.25 76.53 0)
-			(show_name no)
-			(do_not_autoplace no)
-			(effects
-				(font
-					(size 1.27 1.27)
-				)
-				(justify left)
-			)
-		)
-		(property "Footprint" "Resistor_SMD:R_0805_2012Metric"
-			(at 44.45 74.93 0)
-			(hide yes)
-			(show_name no)
-			(do_not_autoplace no)
-			(effects
-				(font
-					(size 1.27 1.27)
-				)
-			)
-		)
-		(property "Datasheet" ""
-			(at 44.45 74.93 0)
-			(hide yes)
-			(show_name no)
-			(do_not_autoplace no)
-			(effects
-				(font
-					(size 1.27 1.27)
-				)
-			)
-		)
-		(property "Description" "Resistor, small symbol"
-			(at 44.45 74.93 0)
-			(hide yes)
-			(show_name no)
-			(do_not_autoplace no)
-			(effects
-				(font
-					(size 1.27 1.27)
-				)
-			)
-		)
-		(property "LCSC" "C17477"
-			(at 44.45 74.93 0)
-			(hide yes)
-			(show_name no)
-			(do_not_autoplace no)
-			(effects
-				(font
-					(size 1.27 1.27)
-				)
-			)
-		)
-		(property "MPN" "0805W8F0000T5E"
-			(at 44.45 74.93 0)
-			(hide yes)
-			(show_name no)
-			(do_not_autoplace no)
-			(effects
-				(font
-					(size 1.27 1.27)
-				)
-			)
-		)
-		(property "Manufacturer" "UNI-ROYAL"
-			(at 44.45 74.93 0)
-			(hide yes)
-			(show_name no)
-			(do_not_autoplace no)
-			(effects
-				(font
-					(size 1.27 1.27)
-				)
-			)
-		)
-		(pin "1"
-		)
-		(pin "2"
-		)
-		(instances
-			(project "Si5351AVFO"
-				(path "/a0000000-0000-4000-8000-000000000001/b0000000-0000-4000-8000-000000000004"
-					(reference "R6")
-					(unit 1)
-				)

Commit message: U1: LCSC C529366 (Si5351A-B-GT, in stock) as primary, C504891 (-GTR) kept as LCSC_ALT
Parts:
- U2: LCSC C504891 -> C529366; LCSC_ALT (none) -> C504891; MPN SI5351A-B-GTR -> SI5351A-B-GT
Changed lines of the file:
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@@
 			)
 		)
-		(property "LCSC" "C504891"
+		(property "LCSC" "C529366"
 			(at 139.7 95.25 0)
 			(hide yes)
@@
 			)
 		)
-		(property "MPN" "SI5351A-B-GTR"
+		(property "LCSC_ALT" "C504891"
 			(at 139.7 95.25 0)
 			(hide yes)
+			(show_name no)
+			(do_not_autoplace no)
+			(effects
+				(font
+					(size 1.27 1.27)
+				)
+			)
+		)
+		(property "MPN" "SI5351A-B-GT"
+			(at 139.7 95.25 0)
+			(hide yes)
